Commit message: CR12A 替换：模型/关节限位、全零位 home、向前重算扫描轨迹、调快节拍
机械臂替换
- 新增 urdf/cr12_macro.xacro：Dobot 官方 DOBOT_6Axis_ROS2_V4 的 CR12 URDF 移植，
  去掉 dummy_link，补 tool0/flange，参数化 prefix
- 新增 meshes/cr12/{base_link0,j1..j6}.ply
- workcell.xacro / workcell.srdf / controllers.yaml / *.rviz 关节名与链同步
- 关节限位由官方 ±6.28 收窄到 ±π（J3 保持 ±2.79），避免解空间炸开

home 位统一为全零位
- 扫描从零位启动并回到零位，打磨接着从零位开始
- 同步 4 处定义：start.launch.xml 的 home_state_joint_positions、
  test.launch.xml 的 zeros.jointN、ros2_control.xacro 的 initial_value、
  scan_traj.yaml 的首尾点

扫描轨迹重算
- 原 8 个航点仍是 HC10 关节值，FK 核算后 tool0 落在 X -0.38~-0.52（基座后方），
  而工件在 X 0.66~0.94（正前方）
- 由 calibration.yaml 反解出相机光轴在法兰系指向 +X，据此以「相机垂直朝下」为约束，
  用 FK + DLS 逆解重算 8 个航点（残差 <1e-4），覆盖坐面上方 Z=0.42、X 0.68~0.90

节拍
- 扫描 60s -> 13.2s
- 打磨 TCP 0.05 -> 0.15 m/s，加速度 0.1 -> 0.5 m/s^2，并提为 launch 参数

Docker
- compose.sim.yml 补 urdf/ 挂载，本地改 URDF 才生效

文档
- README.md 改写为本次替换的过程总结
- 原 README 内容移至 docs/zhixingceng_seat_polishing.md
- .gitignore 忽略 CR12 官方 STL 与网格中间产物、RViz 运行期缓存

遗留：工件当前为坐面坐板，后续需换回原本的半圆工件；
相机标定与打磨头支架仍为 HC10 时代的旧值。

Co-Authored-By: Claude <noreply@anthropic.com>

File: urdf/ros2_control.xacro (robot description, xacro)
@@ -8,83 +8,91 @@
         </xacro:if>
       </hardware>
-      <joint name="${prefix}joint_1_s">
+      <joint name="${prefix}joint1">
         <command_interface name="position">
-          <param name="min">${radians(-180)}</param>
-          <param name="max">${radians(180)}</param>
+          <param name="min">-3.14159265</param>
+          <param name="max">3.14159265</param>
         </command_interface>
         <command_interface name="velocity">
-          <param name="min">${radians(-130)}</param>
-          <param name="max">${radians(130)}</param>
-        </command_interface>
-        <command_interface name="acceleration"/>
-        <state_interface name="position"/>
-        <state_interface name="velocity"/>
-      </joint>
-      <joint name="${prefix}joint_2_l">
-        <command_interface name="position">
-          <param name="min">${radians(-180)}</param>
-          <param name="max">${radians(180)}</param>
-        </command_interface>
-        <command_interface name="velocity">
-          <param name="min">${radians(-130)}</param>
-          <param name="max">${radians(130)}</param>
-        </command_interface>
-        <command_interface name="acceleration"/>
-        <state_interface name="position"/>
-        <state_interface name="velocity"/>
-      </joint>
-      <joint name="${prefix}joint_3_u">
-        <command_interface name="position">
-          <param name="min">${radians(-5)}</param>
-          <param name="max">${radians(355)}</param>
-        </command_interface>
-        <command_interface name="velocity">
-          <param name="min">${radians(-180)}</param>
-          <param name="max">${radians(180)}</param>
+          <param name="min">-3.14</param>
+          <param name="max">3.14</param>
         </command_interface>
         <command_interface name="acceleration"/>
         <state_interface name="position">
-          <param name="initial_value">${radians(90)}</param>
+          <param name="initial_value">0.0</param>
+        </state_interface>
+        <state_interface name="velocity"/>
+      </joint>
+      <joint name="${prefix}joint2">
+        <command_interface name="position">
+          <param name="min">-3.14159265</param>
+          <param name="max">3.14159265</param>
+        </command_interface>
+        <command_interface name="velocity">
+          <param name="min">-3.14</param>
+          <param name="max">3.14</param>
+        </command_interface>
+        <command_interface name="acceleration"/>
+        <state_interface name="position">
+          <param name="initial_value">0.0</param>
+        </state_interface>
+        <state_interface name="velocity"/>
+      </joint>
+      <joint name="${prefix}joint3">
+        <command_interface name="position">
+          <param name="min">-2.79</param>
+          <param name="max">2.79</param>
+        </command_interface>
+        <command_interface name="velocity">
+          <param name="min">-3.89</param>
+          <param name="max">3.89</param>
+        </command_interface>
+        <command_interface name="acceleration"/>
+        <state_interface name="position">
+          <param name="initial_value">0.0</param>
         </state_interface>
         <state_interface name="velocity" />
       </joint>
-      <joint name="${prefix}joint_4_r">
+      <joint name="${prefix}joint4">
         <command_interface name="position">
-          <param name="min">${radians(-180)}</param>
-          <param name="max">${radians(180)}</param>
+          <param name="min">-3.14159265</param>
+          <param name="max">3.14159265</param>
         </command_interface>
         <command_interface name="velocity">
-          <param name="min">${radians(-180)}</param>
-          <param name="max">${radians(180)}</param>
-        </command_interface>
-        <command_interface name="acceleration"/>
-        <state_interface name="position"/>
-        <state_interface name="velocity"/>
-      </joint>
-      <joint name="${prefix}joint_5_b">
-        <command_interface name="position">
-          <param name="min">${radians(-180)}</param>
-          <param name="max">${radians(180)}</param>
-        </command_interface>
-        <command_interface name="velocity">
-          <param name="min">${radians(-250)}</param>
-          <param name="max">${radians(250)}</param>
-        </command_interface>
-        <command_interface name="acceleration"/>
-        <state_interface name="position"/>
-        <state_interface name="velocity"/>
-      </joint>
-      <joint name="${prefix}joint_6_t">
-        <command_interface name="position">
-          <param name="min">${radians(-180)}</param>
-          <param name="max">${radians(180)}</param>
-        </command_interface>
-        <command_interface name="velocity">
-          <param name="min">${radians(-250)}</param>
-          <param name="max">${radians(250)}</param>
+          <param name="min">-3.89</param>
+          <param name="max">3.89</param>
         </command_interface>
         <command_interface name="acceleration"/>
         <state_interface name="position">
-          <param name="initial_value">0.785</param>
+          <param name="initial_value">0.0</param>
+        </state_interface>
+        <state_interface name="velocity"/>
+      </joint>
+      <joint name="${prefix}joint5">
+        <command_interface name="position">
+          <param name="min">-3.14159265</param>
+          <param name="max">3.14159265</param>
+        </command_interface>
+        <command_interface name="velocity">
+          <param name="min">-3.89</param>
+          <param name="max">3.89</param>
+        </command_interface>
+        <command_interface name="acceleration"/>
+        <state_interface name="position">
+          <param name="initial_value">0.0</param>
+        </state_interface>
+        <state_interface name="velocity"/>
+      </joint>
+      <joint name="${prefix}joint6">
+        <command_interface name="position">
+          <param name="min">-3.14159265</param>
+          <param name="max">3.14159265</param>
+        </command_interface>
+        <command_interface name="velocity">
+          <param name="min">-3.89</param>
+          <param name="max">3.89</param>
+        </command_interface>
+        <command_interface name="acceleration"/>
+        <state_interface name="position">
+          <param name="initial_value">0.0</param>
         </state_interface>
         <state_interface name="velocity"/>

File: urdf/workcell.xacro (robot description, xacro)
@@ -1,6 +1,6 @@
 <?xml version="1.0" ?>
-<robot name="motoman_hc10" xmlns:xacro="http://ros.org/wiki/xacro" xmlns:tesseract="https://github.com/tesseract-robotics/tesseract" tesseract:make_convex="true">
-  <xacro:include filename="$(find motoman_hc10_support)/urdf/hc10dt_macro.xacro" />
-  <xacro:motoman_hc10dt prefix=""/>
+<robot name="cr12_robot" xmlns:xacro="http://ros.org/wiki/xacro" xmlns:tesseract="https://github.com/tesseract-robotics/tesseract" tesseract:make_convex="true">
+  <xacro:include filename="cr12_macro.xacro" />
+  <xacro:dobot_cr12 prefix=""/>
   <xacro:include filename="$(find snp_automate_2023)/urdf/ros2_control.xacro"/>
   <xacro:snp_ros2_control name="snp_ros2_control" prefix=""/>
@@ -62,4 +62,5 @@
     <parent link="table"/>
     <child link="base_link"/>
+    <!-- CR12 机械臂相对工作台的位置（可能需要后续微调） -->
     <origin xyz="-0.61 0 0.723" rpy="0 0 0"/>
   </joint>
